File: ScratchBotVer2.0/PCBDesign/scratchBotV2.brd (EAGLE design)
At the start: 100 x 81.3 mm, 38 parts, among them T1 BD139, T3 BD139

Commit message: lI ION BATTERY ADDED AND REVIEW OF OTHER COMPONENTS.
Parts:
- removed CHARGER: BATTERY-CHARGER-LI-PROT, diy-modules:BATTERY-CHARGER-LI-PROT
- removed LI-IONBATTERY: BK-18650-PC2, BK-18650-PC2:BAT_BK-18650-PC2
- added BT1: 1048P, 1048P:BAT_1048P
Connections:
- removed net N$3: CHARGER.B+, LI-IONBATTERY.-
- removed net N$32: CHARGER.OUT+, SW2.2, SWITCH.1
- net N$1: now also BT1.1-, SW2.2, SWITCH.1; no longer CHARGER.B-, LI-IONBATTERY.+
- net N$6: now also BT1.1+; no longer CHARGER.OUT-
Routing:
- net N$32: track 155.9 -> 0.00 mm, vias 5 -> 0
- net N$1: track 100.5 -> 146.4 mm, vias 2 -> 5
- net N$3: track 27.9 -> 0.00 mm
- net N$6: track 81.2 -> 68.3 mm

Commit message: updated
Parts:
- removed BOOSTER: DC-DC-STEP-UP-MT3608, diy-modules:DC-DC-STEP-UP-MT3608
- added LDR: JST-XH-02-PIN-LONG-PAD, Rembrandt Electronics - JST XH Connectors v1-0:JST-XH-02-PACKAGE-LONG-PAD
- added LED1: (no value), adafruit:CHIPLED_1206
- added R1: 10K, bourns:3362H
- added R3: (no value), bourns:3362H
- added R4, R6, R7: 10K, adafruit:M1206
- added R5: (no value), adafruit:M1206
- added SERVO: SERVO, Rembrandt Electronics - JST XH Connectors v1-0 (1):JST-XH-03-PACKAGE-LONG-PAD
- added T2, T4, T5: (no value), transistor:SOT23-EBC
- added U1, U2: LM358M/NOPB, LM358M_NOPB:SOIC127P599X175-8N
Connections:
- new net N$26: LDR.1, R4.2
- new net N$27: R6.1, U1.1
- new net N$3: R1.2, U1.2
- new net N$31: R6.2, T2.B
- new net N$32: LED1.C, T2.C
- new net N$38: LED1.A, R7.1
- new net V+: U2.8
- net 9V-MT3608: no longer BOOSTER.OUT+
- net GND: now also R1.1, R4.1, T2.E, U1.4, U2.4; no longer BOOSTER.OUT-
- net N$18: no longer BOOSTER.IN+
- net N$6: no longer BOOSTER.IN-
- net VCC: now also LDR.2, R1.3, R7.2, U1.8
Routing:
- net N$6: track 68.3 -> 27.9 mm
- net N$18: track 192.2 -> 171.6 mm
- net GND: track 409.7 -> 405.3 mm
- net 9V-MT3608: track 130.2 -> 126.4 mm

Commit message: updated pin number
Parts:
- removed D1: 1N4004, adafruit:DO41-10
- removed LDR/TNKR: LDR/TNKR, Rembrandt Electronics - JST XH Connectors v1-0 (1):JST-XH-03-PACKAGE-LONG-PAD
- removed OUT1-J1: (no value), SparkFun-Connectors:1X02
Connections:
- removed net IR1: ARD_NANO.20, IR1.2, J4.5
- removed net N$24: ARD_NANO.6, J3.6, LDR/TNKR.2
- removed net N$28: D1.A, OUT1-J1.2, R2.1
- removed net N$30: D1.C, OUT1.1
- new net N$39: ARD_NANO.20, DRIVER.7, J4.5
- new net N$40: IR2.2
- new net N$41: ARD_NANO.7, J3.7
- net ECHO: now also ARD_NANO.8, I2C.3, J3.8; no longer ARD_NANO.7, J3.7
- net GND: now also SERVO.3; no longer LDR/TNKR.3
- net IR2: now also DRIVER.1; no longer IR2.2
- net M1B: now also DRIVER.9; no longer DRIVER.7
- net N$10: no longer DRIVER.1
- net N$13: now also BT.4; no longer DRIVER.9
- net N$15: now also ARD_NANO.5, J3.5; no longer ARD_NANO.8, I2C.3, J3.8
- net N$16: now also ARD_NANO.6, J3.6; no longer ARD_NANO.9, I2C.2, J3.9
- net N$23: now also ARD_NANO.9, I2C.2, J3.9; no longer ARD_NANO.5, J3.5
- net N$5: now also SERVO.1; no longer LEDMATRIX.3
- net TX: now also LEDMATRIX.3; no longer BT.4
- net VCC: now also SERVO.2; no longer LDR/TNKR.1, OUT1-J1.1
Routing:
- net N$24: track 126.2 -> 0.00 mm, vias 3 -> 0
- net IR1: track 96.2 -> 0.00 mm
- net N$23: track 131.3 -> 214.6 mm, vias 1 -> 3
- net N$15: track 84.7 -> 4.34 mm, vias 1 -> 0
- net N$13: track 83.2 -> 3.81 mm, vias 2 -> 0
- net ECHO: track 102.4 -> 180.3 mm, vias 1 -> 2
- net M1B: track 86.2 -> 161.9 mm, vias 1 -> 3
- net N$28: track 67.4 -> 0.00 mm, vias 2 -> 0
- net N$30: track 63.0 -> 0.00 mm, vias 3 -> 0
- net N$16: track 91.4 -> 124.9 mm, vias 2 -> 3
- net VCC: track 313.6 -> 301.4 mm
- net N$41: track 0.00 -> 4.34 mm
- net N$39: track 0.00 -> 3.81 mm
- net IR2: track 129.1 -> 125.9 mm
- net TX: track 40.9 -> 39.7 mm
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
Commit message: Two TCR5000  circuit added for line follower.
Parts:
- added LED2, LED3: (no value), adafruit:CHIPLED_1206
- added R10, R11: 10K, adafruit:M1206
- added R8, R9: (no value), adafruit:M1206
- added U3, U4: TCRT5000, TCRT5000:OPTO_TCRT5000
- R5: device adafruit:M1206 -> bourns:3362H
- moved R5 69.1 mm to (-71.1, -151.1)
Connections:
- removed net V+: U2.8
- new net N$24: R8.1, U3.A
- new net N$28: R9.1, U4.A
- new net N$30: LED2.C, T4.C
- new net N$42: R3.2, U2.2
- new net N$43: LED3.A, R11.1
- new net N$44: LED2.A, R10.1
- new net N$45: T4.B, U2.1
- new net N$46: LED3.C, T5.C
- new net N$47: T5.B, U2.7
- new net N$48: R5.2, U2.6
- net GND: now also R3.1, R5.1, T4.E, T5.E, U3.CATH, U3.E, U4.CATH, U4.E
- net N$16: now also U2.3, U3.COLL
- net N$41: now also U2.5, U4.COLL
- net VCC: now also R10.2, R11.2, R3.3, R5.3, R8.2, R9.2, U2.8
Routing:
- net 9V-MT3608: track 126.4 -> 121.0 mm

Commit message: Output Pins of TCR5000 and LDR is connected to the analog pin of Arduino and reviewed the circuit.
Parts:
- removed IR1: IR1, Rembrandt Electronics - JST XH Connectors v1-0 (1):JST-XH-03-PACKAGE-LONG-PAD
- removed IR2: IR2, Rembrandt Electronics - JST XH Connectors v1-0 (1):JST-XH-03-PACKAGE-LONG-PAD
- removed OUT1: A1, Rembrandt Electronics - JST XH Connectors v1-0 (1):JST-XH-02-PACKAGE-LONG-PAD
- added LED4: (no value), adafruit:CHIPLED_1206
Connections:
- removed net N$30: LED2.C, T4.C
- removed net N$40: IR2.2
- removed net N$41: ARD_NANO.7, J3.7, U2.5, U4.COLL
- removed net N$46: LED3.C, T5.C
- new net N$49: LED4.A, R2.1
- net GND: no longer IR1.3, IR2.3
- net N$15: now also ARD_NANO.7, J3.7, LED1.C, T2.C; no longer ARD_NANO.5, J3.5
- net N$16: now also ARD_NANO.5, J3.5, LED3.C, T5.C; no longer ARD_NANO.6, J3.6
- net N$17: now also LED4.C; no longer OUT1.2
- net N$32: now also ARD_NANO.6, J3.6, LED2.C, T4.C, U2.5, U4.COLL; no longer LED1.C, T2.C
- net VCC: no longer IR1.1, IR2.1
Routing:
- net N$32: track 0.00 -> 124.9 mm, vias 0 -> 3
- net N$16: track 124.9 -> 4.34 mm, vias 3 -> 0
- net VCC: track 301.4 -> 293.7 mm
- net N$41: track 4.34 -> 0.00 mm
- net GND: track 404.1 -> 399.8 mm
- net N$17: track 35.3 -> 34.1 mm

Commit message: Resistors value updated
Parts:
- R10, R11: value 10K -> 100E
- R3, R5: value (none) -> 10K
- R7: value 10K -> 330 ohm
- R8, R9: value (none) -> 150 ohm
Changed lines of the file:
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@@
 <attribute name="VALUE" x="-27.4066" y="-83.312" size="1.27" layer="27" ratio="10"/>
 </element>
-<element name="R3" library="bourns" package="3362H" value="" x="-33.02" y="-77.47" smashed="yes">
+<element name="R3" library="bourns" package="3362H" value="10K" x="-33.02" y="-77.47" smashed="yes">
 <attribute name="NAME" x="-36.322" y="-74.168" size="1.27" layer="25" ratio="10"/>
 <attribute name="VALUE" x="-36.2966" y="-83.312" size="1.27" layer="27" ratio="10"/>
@@
 <attribute name="VALUE" x="-38.1" y="-125.73" size="1.27" layer="27" rot="R90"/>
 </element>
-<element name="R7" library="adafruit" package="M1206" value="10K" x="-40.64" y="-130.81" smashed="yes">
+<element name="R7" library="adafruit" package="M1206" value="330 ohm" x="-40.64" y="-130.81" smashed="yes">
 <attribute name="NAME" x="-41.91" y="-129.54" size="1.27" layer="25"/>
 <attribute name="VALUE" x="-41.91" y="-133.35" size="1.27" layer="27"/>
@@
 <attribute name="VALUE" x="-65.91081875" y="-132.35271875" size="1.27676875" layer="27" ratio="10"/>
 </element>
-<element name="R8" library="adafruit" package="M1206" value="" x="-63.5" y="-137.16" smashed="yes">
+<element name="R8" library="adafruit" package="M1206" value="150 ohm" x="-63.5" y="-137.16" smashed="yes">
 <attribute name="NAME" x="-64.77" y="-135.89" size="1.27" layer="25"/>
 <attribute name="VALUE" x="-64.77" y="-139.7" size="1.27" layer="27"/>
 </element>
-<element name="R9" library="adafruit" package="M1206" value="" x="-63.5" y="-142.24" smashed="yes">
+<element name="R9" library="adafruit" package="M1206" value="150 ohm" x="-63.5" y="-142.24" smashed="yes">
 <attribute name="NAME" x="-64.77" y="-140.97" size="1.27" layer="25"/>
 <attribute name="VALUE" x="-64.77" y="-144.78" size="1.27" layer="27"/>
@@
 <attribute name="VALUE" x="-60.96" y="-149.86" size="1.27" layer="27" rot="R90"/>
 </element>
-<element name="R10" library="adafruit" package="M1206" value="10K" x="-59.69" y="-147.32" smashed="yes">
+<element name="R10" library="adafruit" package="M1206" value="100E" x="-59.69" y="-147.32" smashed="yes">
 <attribute name="NAME" x="-60.96" y="-146.05" size="1.27" layer="25"/>
 <attribute name="VALUE" x="-60.96" y="-149.86" size="1.27" layer="27"/>
@@
 <attribute name="VALUE" x="-60.96" y="-156.21" size="1.27" layer="27" rot="R90"/>
 </element>
-<element name="R11" library="adafruit" package="M1206" value="10K" x="-59.69" y="-154.94" smashed="yes">
+<element name="R11" library="adafruit" package="M1206" value="100E" x="-59.69" y="-154.94" smashed="yes">
 <attribute name="NAME" x="-60.96" y="-153.67" size="1.27" layer="25"/>
 <attribute name="VALUE" x="-60.96" y="-157.48" size="1.27" layer="27"/>
 </element>
-<element name="R5" library="bourns" package="3362H" value="" x="-71.12" y="-151.13" smashed="yes">
+<element name="R5" library="bourns" package="3362H" value="10K" x="-71.12" y="-151.13" smashed="yes">
 <attribute name="NAME" x="-74.422" y="-147.828" size="1.27" layer="25" ratio="10"/>
 <attribute name="VALUE" x="-74.3966" y="-156.972" size="1.27" layer="27" ratio="10"/>

Commit message: component placement
Parts:
- moved U4 249.5 mm to (94.0, 68.6), flipped to the bottom, turned to 180 degrees
- moved R5 243.4 mm to (48.3, 61.0)
- moved U3 228.5 mm to (94.0, 50.8), flipped to the bottom, turned to 180 degrees
- moved R11 200.2 mm to (45.7, 15.2)
- moved LED4 198.3 mm to (33.0, 8.89), turned to 90 degrees
- moved R9 194.2 mm to (58.4, 8.89), turned to 180 degrees
- moved LED3 192.3 mm to (33.0, 11.4), turned to 90 degrees
- moved R8 186.2 mm to (52.1, 8.89)
- moved R10 185.0 mm to (39.4, 8.89)
- moved LED2 183.7 mm to (26.7, 11.4), turned to 270 degrees
- moved R7 173.0 mm to (52.1, 15.2)
- moved R6 167.7 mm to (58.4, 15.2), turned to 180 degrees
- moved R3 167.1 mm to (48.3, 68.6)
- moved R1 166.5 mm to (55.9, 68.6)
- moved T5 166.0 mm to (71.1, 8.89), turned to 180 degrees
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Routing:
- net GND: track 399.8 -> 174.5 mm, vias 5 -> 0
- net VCC: track 293.7 -> 76.1 mm, vias 5 -> 0
- net N$18: track 171.6 -> 42.2 mm, vias 4 -> 0
- net IR2: track 125.9 -> 3.81 mm
- net N$14: track 114.4 -> 4.34 mm
- net N$5: track 111.5 -> 4.34 mm
- net N$32: track 124.9 -> 29.2 mm, vias 3 -> 0
- net 9V-MT3608: track 121.0 -> 25.7 mm, vias 3 -> 0
- net N$33: track 127.3 -> 39.5 mm, vias 2 -> 0
- net N$23: track 214.6 -> 136.3 mm, vias 3 -> 0
- net ECHO: track 180.3 -> 107.5 mm, vias 2 -> 0
- net N$8: track 100.2 -> 33.8 mm, vias 3 -> 0
- net M1B: track 161.9 -> 100.5 mm, vias 3 -> 0
- net N$21: track 97.8 -> 38.9 mm, vias 1 -> 0
- net N$20: track 104.8 -> 46.7 mm, vias 2 -> 0
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